File: KiCad/ESP32-C3-SuperMini/ESP32-C3-SuperMini.kicad_pcb (KiCad board)
At the start: 2 copper layers, 18 x 22.5 mm, 39 parts, among them J1 USB_C_Receptacle_USB2.0_14P, SW1 SW_Push, SW2 SW_Push, U1 ESP32-C3, U2 ME6211C33M5G, Y1 Crystal_GND24

Commit message: v1
Parts:
- U1: value ESP32-C3 -> ESP32-C3FN4
