File: KiCad/ESP32-C3-SuperMini/ESP32-C3-SuperMini.kicad_sch (KiCad schematic)
At the start: 39 parts, among them J1 USB_C_Receptacle_USB2.0_14P, SW1 SW_Push, SW2 SW_Push, U1 ESP32-C3, U2 ME6211C33M5G, Y1 Crystal_GND24

Commit message: v1
Parts:
- AE1: LCSC (none) -> C89334
- C1, C13, C3, C7: LCSC (none) -> C76934
- C10, C2, C4, C8: LCSC (none) -> C2846675
- C11, C12: LCSC (none) -> C115548
- C14, C15, C5: LCSC (none) -> C315248
- C6: LCSC (none) -> C85893
- C9: LCSC (none) -> C76941
- H1, H2: now left out of the parts list
- L1: LCSC (none) -> C98043
- L2: LCSC (none) -> C77115
- R1, R2, R3, R4: LCSC (none) -> C4332048
- R10, R9: LCSC (none) -> C270355
- R5, R6, R7, R8: LCSC (none) -> C25837
- U1: value ESP32-C3 -> ESP32-C3FN4; LCSC (none) -> C2848860
Connections:
- no-connect marks 0 -> 6
